Commit message: Minor fix.

File: urdf/sick_lms1xx.urdf.xacro (robot description, xacro)
@@ -31,5 +31,5 @@
         <mass value="1.1" />
         <origin xyz="0 0 0" />
-        <inertia ixx="${0.0833333 * mass * (0.102*0.102 + 0.152*0.152)}" ixy="0.0" ixz="0.0"
+        <inertia ixx="${0.0833333 * 1.1 * (0.102*0.102 + 0.152*0.152)}" ixy="0.0" ixz="0.0"
           iyy="${0.0833333 * 1.1 * (0.105*0.105 + 0.152*0.152)}" iyz="0.0"
           izz="${0.0833333 * 1.1 * (0.105*0.105 + 0.102*0.102)}" />

Commit message: Removed underscore after prefix.

File: urdf/sick_lms1xx.urdf.xacro (robot description, xacro)
@@ -27,5 +27,5 @@
 <robot xmlns:xacro="http://ros.org/wiki/xacro">
   <xacro:macro name="sick_lms1xx" params="prefix topic">
-    <link name="${prefix}_laser">
+    <link name="${prefix}laser">
       <inertial>
         <mass value="1.1" />
@@ -49,7 +49,7 @@
       </collision>
     </link>
-    <gazebo reference="${prefix}_laser">
+    <gazebo reference="${prefix}laser">
       <turnGravityOff>true</turnGravityOff>
-      <sensor type="ray" name="${prefix}_laser">
+      <sensor type="ray" name="${prefix}laser">
         <pose>0 0 0 0 0 0</pose>
         <visualize>false</visualize>
@@ -77,5 +77,5 @@
         <plugin name="gazebo_ros_laser" filename="libgazebo_ros_laser.so">
           <topicName>${prefix}/${topic}</topicName>
-          <frameName>${prefix}_laser</frameName>
+          <frameName>${prefix}laser</frameName>
         </plugin>
       </sensor>

Commit message: Updated to only used frame and topic parameters.

File: urdf/sick_lms1xx.urdf.xacro (robot description, xacro)
@@ -26,6 +26,6 @@
 -->
 <robot xmlns:xacro="http://ros.org/wiki/xacro">
-  <xacro:macro name="sick_lms1xx" params="prefix topic">
-    <link name="${prefix}laser">
+  <xacro:macro name="sick_lms1xx" params="frame:=laser topic:=scan" >
+    <link name="${frame}">
       <inertial>
         <mass value="1.1" />
@@ -49,7 +49,7 @@
       </collision>
     </link>
-    <gazebo reference="${prefix}laser">
+    <gazebo reference="${frame}">
       <turnGravityOff>true</turnGravityOff>
-      <sensor type="ray" name="${prefix}laser">
+      <sensor type="ray" name="${frame}">
         <pose>0 0 0 0 0 0</pose>
         <visualize>false</visualize>
@@ -76,6 +76,6 @@
         </ray>
         <plugin name="gazebo_ros_laser" filename="libgazebo_ros_laser.so">
-          <topicName>${prefix}/${topic}</topicName>
-          <frameName>${prefix}laser</frameName>
+          <topicName>${topic}</topicName>
+          <frameName>${frame}</frameName>
         </plugin>
       </sensor>

Commit message: add parameters 'sample_size' and 'update_rate' for gazebo's ray plugin

File: urdf/sick_lms1xx.urdf.xacro (robot description, xacro)
@@ -26,5 +26,5 @@
 -->
 <robot xmlns:xacro="http://ros.org/wiki/xacro">
-  <xacro:macro name="sick_lms1xx" params="frame:=laser topic:=scan" >
+  <xacro:macro name="sick_lms1xx" params="frame:=laser topic:=scan sample_size:=720 update_rate:=50" >
     <link name="${frame}">
       <inertial>
@@ -54,9 +54,9 @@
         <pose>0 0 0 0 0 0</pose>
         <visualize>false</visualize>
-        <update_rate>50</update_rate>
+        <update_rate>${update_rate}</update_rate>
         <ray>
           <scan>
             <horizontal>
-              <samples>720</samples>
+              <samples>${sample_size}</samples>
               <resolution>1</resolution>
               <min_angle>-2.35619</min_angle>

Commit message: Exposed parameters min_range and max_range

File: urdf/sick_lms1xx.urdf.xacro (robot description, xacro)
@@ -26,5 +26,5 @@
 -->
 <robot xmlns:xacro="http://ros.org/wiki/xacro">
-  <xacro:macro name="sick_lms1xx" params="frame:=laser topic:=scan sample_size:=720 update_rate:=50" >
+  <xacro:macro name="sick_lms1xx" params="frame:=laser topic:=scan sample_size:=720 update_rate:=50 min_range:=0.1 max_range:=30.0" >
     <link name="${frame}">
       <inertial>
@@ -65,6 +65,6 @@
           </scan>
           <range>
-            <min>0.10</min>
-            <max>30.0</max>
+            <min>${min_range}</min>
+            <max>${max_range}</max>
             <resolution>0.01</resolution>
           </range>

Commit message: Add robot namespace to lidar plugin

File: urdf/sick_lms1xx.urdf.xacro (robot description, xacro)
@@ -26,5 +26,5 @@
 -->
 <robot xmlns:xacro="http://ros.org/wiki/xacro">
-  <xacro:macro name="sick_lms1xx" params="frame:=laser topic:=scan sample_size:=720 update_rate:=50 min_range:=0.1 max_range:=30.0" >
+  <xacro:macro name="sick_lms1xx" params="frame:=laser topic:=scan sample_size:=720 update_rate:=50 min_range:=0.1 max_range:=30.0 robot_namespace:=/" >
     <link name="${frame}">
       <inertial>
@@ -78,4 +78,5 @@
           <topicName>${topic}</topicName>
           <frameName>${frame}</frameName>
+          <robotNamespace>${robot_namespace}</robotNamespace>
         </plugin>
       </sensor>

Commit message: migration to ros2 foxy

File: urdf/sick_lms1xx.urdf.xacro (robot description, xacro)
@@ -40,5 +40,5 @@
         <geometry>
           <!-- Origin of this mesh is the focal point of the LIDAR. -->
-          <mesh filename="package://lms1xx/meshes/sick-lms1xx.dae" />
+          <mesh filename="file://$(find lms1xx)/meshes/sick-lms1xx.dae" />
         </geometry>
       </visual>
